Commit message: Remove all slider GUI elements and replace with fixed values for robot positions, orientations, and pipe settings

File: rb10_1300e_DDA.urdf (robot description, URDF)
Before this commit: robot dda_rb10_1300e, 9 links, 8 joints
Links:
- link dda_link0: geometry collision mesh filename=./meshes/rb10_1300e/collision/link0.stl; visual mesh filename=./meshes/rb10_1300e/visual/link0.dae
- link dda_link1: geometry collision mesh filename=./meshes/rb10_1300e/collision/link1.stl; visual mesh filename=./meshes/rb10_1300e/visual/link1.dae
- link dda_link2: geometry collision mesh filename=./meshes/rb10_1300e/collision/link2.stl; visual mesh filename=./meshes/rb10_1300e/visual/link2.dae
- link dda_link3: geometry collision mesh filename=./meshes/rb10_1300e/collision/link3.stl; visual mesh filename=./meshes/rb10_1300e/visual/link3.dae
- link dda_link4: geometry collision mesh filename=./meshes/rb10_1300e/collision/link4.stl; visual mesh filename=./meshes/rb10_1300e/visual/link4.dae
- link dda_link5: geometry collision mesh filename=./meshes/rb10_1300e/collision/link5.stl; visual mesh filename=./meshes/rb10_1300e/visual/link5.dae
- link dda_link6: geometry collision mesh filename=./meshes/rb10_1300e/collision/link6.stl; visual mesh filename=./meshes/rb10_1300e/visual/link6.dae
- link dda_link_end: geometry collision mesh filename=./meshes/link_dda.stl scale=0.001 0.001 0.001; visual mesh filename=./meshes/link_dda.stl scale=0.001 0.001 0.001

File: rb10_1300e_RT.urdf (robot description, URDF)
Before this commit: robot rt_rb10_1300e, 9 links, 8 joints
Links:
- link rt_link0: geometry collision mesh filename=./meshes/rb10_1300e/collision/link0.stl; visual mesh filename=./meshes/rb10_1300e/visual/link0.dae
- link rt_link1: geometry collision mesh filename=./meshes/rb10_1300e/collision/link1.stl; visual mesh filename=./meshes/rb10_1300e/visual/link1.dae
- link rt_link2: geometry collision mesh filename=./meshes/rb10_1300e/collision/link2.stl; visual mesh filename=./meshes/rb10_1300e/visual/link2.dae
- link rt_link3: geometry collision mesh filename=./meshes/rb10_1300e/collision/link3.stl; visual mesh filename=./meshes/rb10_1300e/visual/link3.dae
- link rt_link4: geometry collision mesh filename=./meshes/rb10_1300e/collision/link4.stl; visual mesh filename=./meshes/rb10_1300e/visual/link4.dae
- link rt_link5: geometry collision mesh filename=./meshes/rb10_1300e/collision/link5.stl; visual mesh filename=./meshes/rb10_1300e/visual/link5.dae
- link rt_link6: geometry collision mesh filename=./meshes/rb10_1300e/collision/link6.stl; visual mesh filename=./meshes/rb10_1300e/visual/link6.dae
- link rt_link_end: geometry collision mesh filename=./meshes/link_rt.stl scale=0.001 0.001 0.001; visual mesh filename=./meshes/link_rt.stl scale=0.001 0.001 0.001
